Commit message: change urdf
move wheels so their position is closer to how it is on real robot

File: install/iir_base/share/iir_base/urdf/iir_description.urdf.xacro (robot description, xacro)
@@ -24,5 +24,5 @@
     </collision>
     <visual>
-      <origin xyz="0 0 ${base_height/2}" rpy="0 0 0"/>
+      <origin xyz=".22 0 ${base_height/2}" rpy="0 0 0"/>
       <geometry>
         <box size="${base_width} ${base_length} ${base_height}"/>
@@ -44,5 +44,5 @@
       <parent link="base_link"/>
       <child link="left_wheel"/>
-      <origin xyz=".08 .29 ${z_offset}" rpy="0 0 0"/>
+      <origin xyz=".22 .29 ${z_offset}" rpy="0 0 0"/>
       <axis xyz="0 1 0"/>
       <dynamics damping="0.2"/>
@@ -86,5 +86,5 @@
       <parent link="base_link"/>
       <child link="right_wheel"/>
-      <origin xyz=".08 -.29 ${z_offset}" rpy="0 0 0"/>
+      <origin xyz=".22 -.29 ${z_offset}" rpy="0 0 0"/>
       <axis xyz="0 1 0"/>
       <dynamics damping="0.2"/>

File: src/IIR_base/urdf/iir_description.urdf.xacro (robot description, xacro)
@@ -44,5 +44,5 @@
       <parent link="base_link"/>
       <child link="left_wheel"/>
-      <origin xyz=".08 .29 ${z_offset}" rpy="0 0 0"/>
+      <origin xyz=".22 .29 ${z_offset}" rpy="0 0 0"/>
       <axis xyz="0 1 0"/>
       <dynamics damping="0.2"/>
@@ -86,5 +86,5 @@
       <parent link="base_link"/>
       <child link="right_wheel"/>
-      <origin xyz=".08 -.29 ${z_offset}" rpy="0 0 0"/>
+      <origin xyz=".22 -.29 ${z_offset}" rpy="0 0 0"/>
       <axis xyz="0 1 0"/>
       <dynamics damping="0.2"/>

Commit message: update URDF
move the position of base link so that it is closer to the pivot point (in between the driven wheels)

File: install/iir_base/share/iir_base/urdf/iir_description.urdf.xacro (robot description, xacro)
@@ -17,4 +17,5 @@
   <!-- Base Link -->
   <link name="base_link">
+  <origin xyz="-0.1 0 0"/>
     <collision>
       <origin xyz="0 0 ${base_height/2}" rpy="0 0 0"/>
@@ -24,5 +25,5 @@
     </collision>
     <visual>
-      <origin xyz=".22 0 ${base_height/2}" rpy="0 0 0"/>
+      <origin xyz="-.15 0 ${base_height/2}" rpy="0 0 0"/>
       <geometry>
         <box size="${base_width} ${base_length} ${base_height}"/>

File: src/IIR_base/urdf/iir_description.urdf.xacro (robot description, xacro)
@@ -17,4 +17,5 @@
   <!-- Base Link -->
   <link name="base_link">
+  <origin xyz="-0.1 0 0"/>
     <collision>
       <origin xyz="0 0 ${base_height/2}" rpy="0 0 0"/>
@@ -24,5 +25,5 @@
     </collision>
     <visual>
-      <origin xyz="0 0 ${base_height/2}" rpy="0 0 0"/>
+      <origin xyz="-.15 0 ${base_height/2}" rpy="0 0 0"/>
       <geometry>
         <box size="${base_width} ${base_length} ${base_height}"/>

Commit message: update

File: install/iir_base/share/iir_base/urdf/iir_description.urdf.xacro (robot description, xacro)
@@ -17,7 +17,7 @@
   <!-- Base Link -->
   <link name="base_link">
-  <origin xyz="-0.1 0 0"/>
+  <origin xyz="-0.13 0 0"/>
     <collision>
-      <origin xyz="0 0 ${base_height/2}" rpy="0 0 0"/>
+      <origin xyz="-.13 0 ${base_height/2}" rpy="0 0 0"/>
       <geometry>
         <box size="${base_width} ${base_length} ${base_height}"/>
@@ -45,5 +45,5 @@
       <parent link="base_link"/>
       <child link="left_wheel"/>
-      <origin xyz="0 .29 ${z_offset}" rpy="0 0 0"/>
+      <origin xyz="0 .254 ${z_offset}" rpy="0 0 0"/>
       <axis xyz="0 1 0"/>
       <dynamics damping="0.2"/>
@@ -87,5 +87,5 @@
       <parent link="base_link"/>
       <child link="right_wheel"/>
-      <origin xyz="0 -.29 ${z_offset}" rpy="0 0 0"/>
+      <origin xyz="0 -.254 ${z_offset}" rpy="0 0 0"/>
       <axis xyz="0 1 0"/>
       <dynamics damping="0.2"/>

File: src/IIR_base/urdf/iir_description.urdf.xacro (robot description, xacro)
@@ -45,5 +45,5 @@
       <parent link="base_link"/>
       <child link="left_wheel"/>
-      <origin xyz="0 .29 ${z_offset}" rpy="0 0 0"/>
+      <origin xyz="0 .254 ${z_offset}" rpy="0 0 0"/>
       <axis xyz="0 1 0"/>
       <dynamics damping="0.2"/>
@@ -87,5 +87,5 @@
       <parent link="base_link"/>
       <child link="right_wheel"/>
-      <origin xyz="0 -.29 ${z_offset}" rpy="0 0 0"/>
+      <origin xyz="0 -.254 ${z_offset}" rpy="0 0 0"/>
       <axis xyz="0 1 0"/>
       <dynamics damping="0.2"/>

Commit message: idk what to cal this

File: install/iir_base/share/iir_base/urdf/iir_description.urdf.xacro (robot description, xacro)
@@ -74,4 +74,13 @@
         </inertial>
       </link>
+<transmission name="left_wheel_trans">
+  <type>transmission_interface/SimpleTransmission</type>
+  <actuator name="left_motor">
+    <mechanicalReduction>11.111</mechanicalReduction>
+  </actuator>
+  <joint name="left_wheel_joint">
+    <hardwareInterface>hardware_interface/VelocityJointInterface</hardwareInterface>
+  </joint>
+</transmission>
     <gazebo reference="left_wheel">
       <mu1>1.0</mu1>
@@ -126,4 +135,13 @@
       <material>Gazebo/DarkGrey</material>
     </gazebo>
+<transmission name="right_wheel_trans">
+  <type>transmission_interface/SimpleTransmission</type>
+  <actuator name="right_motor">
+    <mechanicalReduction>11.111</mechanicalReduction>
+  </actuator>
+  <joint name="right_wheel_joint">
+    <hardwareInterface>hardware_interface/VelocityJointInterface</hardwareInterface>
+  </joint>
+</transmission>
     <!-- <joint name="caster_frontal_wheel_joint" type="fixed">
       <parent link="base_link"/>

File: install/iir_base/share/iir_base/urdf/iirbot.ros2_control.xacro (robot description, xacro)
@@ -13,23 +13,37 @@
         <hardware>
            <!-- <plugin>mock_components/GenericSystem</plugin> -->
-           <plugin>topic_based_ros2_control/TopicBasedSystem</plugin>
-           <param name="joint_commands_topic">/joint_ctrl</param> <!-- this is the publisher-->
-           <param name="joint_states_topic">/wheelmux</param> <!-- this is the subscriber-->
-           <param name="sum_wrapped_joint_states">true</param>
-           <param name="trigger_joint_command_threshold">-1</param>
-           <param name="calculate_dynamics">true</param>
+                  <plugin>odrive_ros2_control_plugin/ODriveHardwareInterface</plugin>
+          <param name="can">can0</param>
           </hardware>
       </xacro:if>
       <joint name="left_wheel_joint">
+	             <param name="node_id">16</param>
+        <command_interface name="velocity"/>
+        <state_interface name="position"/>
+        <state_interface name="velocity"/>
+</joint>
+      <joint name="right_wheel_joint">
+	              <param name="node_id">19</param>
         <command_interface name="velocity"/>
         <state_interface name="position"/>
         <state_interface name="velocity"/>
       </joint>
-      <joint name="right_wheel_joint">
-        <command_interface name="velocity"/>
-        <state_interface name="position"/>
-        <state_interface name="velocity"/>
-      </joint>
-    </ros2_control>
+ <transmission name="transmission1">
+        <plugin>transmission_interface/SimpleTransmission</plugin>
+        <actuator name="actuator1" role="actuator1"/>
+        <joint name="left_wheel_joint" role="left_wheel_joint">
+          <mechanical_reduction>11.111111</mechanical_reduction>
+          <offset>0.0</offset>
+        </joint>
+      </transmission>
+ <transmission name="transmission2">
+        <plugin>transmission_interface/SimpleTransmission</plugin>
+        <actuator name="actuator2" role="actuator2"/>
+        <joint name="right_wheel_joint" role="right_wheel_joint">
+          <mechanical_reduction>11.111111</mechanical_reduction>
+          <offset>0.0</offset>
+        </joint>
+      </transmission>
+</ros2_control>
 <gazebo>
   <plugin filename="libgz_ros2_control-system.so" name="gz_ros2_control::GazeboSimROS2ControlPlugin">
@@ -44,5 +58,5 @@
   <!-- kinematics -->
   <wheel_separation>.508</wheel_separation>
-  <wheel_radius>0.0635</wheel_radius> <!-- computed from <wheel_diameter> in the original plugin-->
+  <wheel_radius>0.05715</wheel_radius> <!-- computed from <wheel_diameter> in the original plugin-->
   <!-- limits -->
   <max_linear_acceleration>100</max_linear_acceleration> <!-- computed from <max_linear_acceleration> in the original plugin-->

Commit message: add base_footprint link
nesc for the joint to work properly

File: install/iir_base/share/iir_base/urdf/iir_description.urdf.xacro (robot description, xacro)
@@ -174,4 +174,10 @@
       </link>
       -->
+      <link name="base_footprint" />
+    <joint name="base_link_joint" type="fixed">
+  <parent link="base_footprint"/>
+  <child link="base_link"/>
+  <origin xyz="0 0 0.05" rpy="0 0 0"/>
+</joint>
     <joint name="caster_rear_wheel_joint" type="fixed">
       <parent link="base_link"/>

File: src/IIR_base/urdf/iir_description.urdf.xacro (robot description, xacro)
@@ -174,4 +174,5 @@
       </link>
       -->
+      <link name="base_footprint" />
     <joint name="base_link_joint" type="fixed">
   <parent link="base_footprint"/>

Commit message: apply description and radius updates

File: install/iir_base/share/iir_base/urdf/iir_description.urdf.xacro (robot description, xacro)
@@ -5,13 +5,13 @@
   <xacro:property name="PI" value="3.1415926535897931"/>
   <xacro:property name="base_mass" value="0.3" /> <!-- arbitrary value for base mass -->
-  <xacro:property name="base_width" value=".63" />
-  <xacro:property name="base_length" value=".57" />
-  <xacro:property name="base_height" value="0.17" />
+  <xacro:property name="base_width" value=".512" />
+  <xacro:property name="base_length" value=".5334" />
+  <xacro:property name="base_height" value="0.25" />
   <xacro:property name="wheel_mass" value="0.3" /> <!-- arbitrary value for wheel mass -->
   <xacro:property name="wheel_len" value="0.040" />
-  <!-- wheels are .5m apart -->
-  <xacro:property name="wheel_radius" value="0.0635" />
+  <!-- wheels are .362m apart -->
+  <xacro:property name="wheel_radius" value="0.0835" />
   <xacro:property name="caster_wheel_mass" value="0.1" /> <!-- arbitrary value for caster wheel mass -->
-  <xacro:property name="caster_wheel_radius" value="0.042" />
+  <xacro:property name="caster_wheel_radius" value="0.0835" />
   <xacro:property name="z_offset" value="-${base_height/3}" /> <!-- Space btw top of beam and the each joint -->
   <!-- Base Link -->
@@ -32,5 +32,5 @@
     </visual>
     <inertial>
-      <origin xyz="0 0 0" rpy="0 0 0"/>
+      <origin xyz="-.18 0 0" rpy="-.18 0 0"/>
       <mass value="${base_mass}"/>
       <inertia

File: src/IIR_base/urdf/iir_description.urdf.xacro (robot description, xacro)
@@ -5,13 +5,13 @@
   <xacro:property name="PI" value="3.1415926535897931"/>
   <xacro:property name="base_mass" value="0.3" /> <!-- arbitrary value for base mass -->
-  <xacro:property name="base_width" value=".63" />
-  <xacro:property name="base_length" value=".57" />
-  <xacro:property name="base_height" value="0.17" />
+  <xacro:property name="base_width" value=".512" />
+  <xacro:property name="base_length" value=".5334" />
+  <xacro:property name="base_height" value="0.25" />
   <xacro:property name="wheel_mass" value="0.3" /> <!-- arbitrary value for wheel mass -->
   <xacro:property name="wheel_len" value="0.040" />
-  <!-- wheels are .5m apart -->
-  <xacro:property name="wheel_radius" value="0.0635" />
+  <!-- wheels are .362m apart -->
+  <xacro:property name="wheel_radius" value="0.0835" />
   <xacro:property name="caster_wheel_mass" value="0.1" /> <!-- arbitrary value for caster wheel mass -->
-  <xacro:property name="caster_wheel_radius" value="0.042" />
+  <xacro:property name="caster_wheel_radius" value="0.0835" />
   <xacro:property name="z_offset" value="-${base_height/3}" /> <!-- Space btw top of beam and the each joint -->
   <!-- Base Link -->
@@ -32,5 +32,5 @@
     </visual>
     <inertial>
-      <origin xyz="0 0 0" rpy="0 0 0"/>
+      <origin xyz="-.18 0 0" rpy="0 0 0"/>
       <mass value="${base_mass}"/>
       <inertia

Commit message: add ekf for 1 imu, add 2 imu links.
make sure to check orientation when
mounting is done

File: install/iir_base/share/iir_base/urdf/iir_description.urdf.xacro (robot description, xacro)
@@ -5,11 +5,11 @@
   <xacro:property name="PI" value="3.1415926535897931"/>
   <xacro:property name="base_mass" value="0.3" /> <!-- arbitrary value for base mass -->
-  <xacro:property name="base_width" value=".63" />
-  <xacro:property name="base_length" value=".57" />
+  <xacro:property name="base_width" value=".55" />
+  <xacro:property name="base_length" value=".51" />
   <xacro:property name="base_height" value="0.17" />
   <xacro:property name="wheel_mass" value="0.3" /> <!-- arbitrary value for wheel mass -->
   <xacro:property name="wheel_len" value="0.040" />
   <!-- wheels are .5m apart -->
-  <xacro:property name="wheel_radius" value="0.0635" />
+  <xacro:property name="wheel_radius" value="0.0825" />
   <xacro:property name="caster_wheel_mass" value="0.1" /> <!-- arbitrary value for caster wheel mass -->
   <xacro:property name="caster_wheel_radius" value="0.042" />
@@ -74,13 +74,36 @@
         </inertial>
       </link>
-<transmission name="left_wheel_trans">
-  <type>transmission_interface/SimpleTransmission</type>
-  <actuator name="left_motor">
-    <mechanicalReduction>11.111</mechanicalReduction>
-  </actuator>
-  <joint name="left_wheel_joint">
-    <hardwareInterface>hardware_interface/VelocityJointInterface</hardwareInterface>
-  </joint>
-</transmission>
+ <!-- IMU Link -->
+    <joint name="imu_joint_1" type="fixed">
+      <parent link="base_link"/>
+      <child link="imu_link_1"/>
+      <origin xyz="-0.35 -.20 ${base_height}" rpy="0 0 0"/>
+    </joint>
+    <link name="imu_link_1">
+      <inertial>
+        <origin xyz="0 0 0" rpy="0 0 0"/>
+        <mass value="0.01"/>
+        <inertia
+          ixx="0.0001" ixy="0.0" ixz="0.0"
+          iyy="0.0001" iyz="0.0"
+          izz="0.0001"/>
+      </inertial>
+    </link>
+ <!-- IMU Link -->
+    <joint name="imu_joint_2" type="fixed">
+      <parent link="base_link"/>
+      <child link="imu_link_2"/>
+      <origin xyz="-0.35 .20 ${base_height}" rpy="0 0 0"/>
+    </joint>
+    <link name="imu_link_2">
+      <inertial>
+        <origin xyz="0 0 0" rpy="0 0 0"/>
+        <mass value="0.01"/>
+        <inertia
+          ixx="0.0001" ixy="0.0" ixz="0.0"
+          iyy="0.0001" iyz="0.0"
+          izz="0.0001"/>
+      </inertial>
+    </link>
     <gazebo reference="left_wheel">
       <mu1>1.0</mu1>

Commit message: Created new launch files for SIM (WIP)

File: install/iir_base/share/iir_base/urdf/iir_description.urdf.xacro (robot description, xacro)
@@ -75,12 +75,12 @@
       </link>
  <!-- IMU Link -->
-    <joint name="imu_joint_1" type="fixed">
-      <parent link="base_link"/>
-      <child link="imu_link_1"/>
-      <origin xyz="-0.35 -.20 ${base_height}" rpy="0 0 0"/>
-    </joint>
-    <link name="imu_link_1">
-      <inertial>
-        <origin xyz="0 0 0" rpy="0 0 0"/>
+    <joint name="imu_joint_0" type="fixed">
+      <parent link="base_link"/>
+      <child link="imu_link_0"/>
+      <origin xyz="-0.35 -.20 ${base_height}" rpy="0 0 ${PI/2}"/>
+    </joint>
+    <link name="imu_link_0">
+      <inertial>
+        <origin xyz="0 0 0" rpy="0 0 ${PI/2}"/>
         <mass value="0.01"/>
         <inertia
@@ -91,12 +91,12 @@
     </link>
  <!-- IMU Link -->
-    <joint name="imu_joint_2" type="fixed">
-      <parent link="base_link"/>
-      <child link="imu_link_2"/>
-      <origin xyz="-0.35 .20 ${base_height}" rpy="0 0 0"/>
-    </joint>
-    <link name="imu_link_2">
-      <inertial>
-        <origin xyz="0 0 0" rpy="0 0 0"/>
+  <joint name="imu_joint_1" type="fixed">
+    <parent link="base_link"/>
+    <child link="imu_link_1"/>
+    <origin xyz="-0.35 .20 ${base_height}" rpy="0 0 ${PI/2}"/>
+  </joint>
+    <link name="imu_link_1">
+      <inertial>
+        <origin xyz="0 0 0" rpy="0 0 ${PI/2}"/>
         <mass value="0.01"/>
         <inertia
@@ -226,4 +226,40 @@
         </inertial>
       </link>
+    <!-- Depth Camera Link -->
+    <joint name="depth_camera_joint" type="fixed">
+      <parent link="base_link"/>
+      <child link="depth_camera_link"/>
+      <origin xyz="0.14 0 ${base_height}" rpy="0 0 0"/>
+    </joint>
+    <link name="depth_camera_link">
+      <visual>
+        <origin xyz="0 0 0" rpy="0 0 0"/>
+        <geometry>
+          <box size="0.025 0.09 0.025"/>
+        </geometry>
+        <material name="black"/>
+      </visual>
+      <collision>
+        <origin xyz="0 0 0" rpy="0 0 0"/>
+        <geometry>
+          <box size="0.025 0.09 0.025"/>
+        </geometry>
+      </collision>
+      <inertial>
+        <origin xyz="0 0 0" rpy="0 0 0"/>
+        <mass value="0.05"/>
+        <inertia
+          ixx="0.0001" ixy="0.0" ixz="0.0"
+          iyy="0.0001" iyz="0.0"
+          izz="0.0001"/>
+      </inertial>
+    </link>
+    <!-- Depth Camera Optical Frame (ROS convention: z forward, x right, y down) -->
+    <joint name="depth_camera_optical_joint" type="fixed">
+      <parent link="depth_camera_link"/>
+      <child link="depth_camera_optical_frame"/>
+      <origin xyz="0 0 0" rpy="${-PI/2} 0 ${-PI/2}"/>
+    </joint>
+    <link name="depth_camera_optical_frame"/>
   </xacro:macro>
 </robot>

File: install/iir_base/share/iir_base/urdf/iirbot.ros2_control.xacro (robot description, xacro)
@@ -3,20 +3,18 @@
   <xacro:macro name="iirbot_ros2_control" params="name prefix use_mock_hardware">
     <ros2_control name="${name}" type="system">
-      <xacro:unless value="${use_mock_hardware}">
+      <xacro:if value="${use_mock_hardware}">
         <hardware>
           <plugin>gz_ros2_control/GazeboSimSystem</plugin>
           <param name="calculate_dynamics">true</param>
-          <!-- having calculate dynamics o -->
         </hardware>
-      </xacro:unless>
-      <xacro:if value="${use_mock_hardware}">
+      </xacro:if>
+      <xacro:unless value="${use_mock_hardware}">
         <hardware>
-          <!-- <plugin>mock_components/GenericSystem</plugin> -->
           <plugin>odrive_ros2_control_plugin/ODriveHardwareInterface</plugin>
           <param name="can">can0</param>
         </hardware>
-      </xacro:if>
+      </xacro:unless>
       <joint name="left_wheel_joint">
-        <param name="node_id">16</param>
+        <param name="node_id">19</param> <!-- ODrive node ID for left wheel -->
         <command_interface name="velocity" />
         <state_interface name="position" />
@@ -24,5 +22,5 @@
       </joint>
       <joint name="right_wheel_joint">
-        <param name="node_id">19</param>
+        <param name="node_id">16</param> <!-- ODrive node ID for right wheel -->
         <command_interface name="velocity" />
         <state_interface name="position" />
