Commit message: try editing urdf - dealing with tf errors

File: src/IIR_base/urdf/hokuyo_ust10.urdf.xacro (robot description, xacro)
@@ -60,6 +60,3 @@
     </gazebo>
   </xacro:macro>
-    <xacro:hokuyo_ust10_mount prefix="" topic="scan" parent_link="base_link" min_angle="-2.35619" max_angle="2.35619">
-  <origin xyz="0 0 0.1" rpy="0 0 0" />
-  </xacro:hokuyo_ust10_mount>
 </robot>

File: src/IIR_base/urdf/iirbot.urdf.xacro (robot description, xacro)
@@ -11,4 +11,7 @@
   <xacro:include filename="$(find iir_base)/urdf/iirbot.ros2_control.xacro" />
   <xacro:iirbot_desc prefix="$(arg prefix)" />
+  <xacro:hokuyo_ust10_mount prefix="" topic="scan" parent_link="base_link" min_angle="-2.35619" max_angle="2.35619">
+  <origin xyz="0 0 0.1" rpy="0 0 0" />
+  </xacro:hokuyo_ust10_mount>
   <xacro:iirbot_ros2_control
     name="IirBot" prefix="$(arg prefix)" use_mock_hardware="$(arg use_mock_hardware)"/>
