Commit message: Additional updates to the URDF

File: src/IIR_base/urdf/iir_description.urdf.xacro (robot description, xacro)
@@ -25,5 +25,5 @@
     </collision>
     <visual>
-      <origin xyz="-.15 0 ${base_height/2}" rpy="0 0 0"/>
+      <origin xyz="-.13 0 ${base_height/2}" rpy="0 0 0"/>
       <geometry>
         <box size="${base_width} ${base_length} ${base_height}"/>
@@ -45,5 +45,5 @@
       <parent link="base_link"/>
       <child link="left_wheel"/>
-      <origin xyz=".22 .29 ${z_offset}" rpy="0 0 0"/>
+      <origin xyz="0 .29 ${z_offset}" rpy="0 0 0"/>
       <axis xyz="0 1 0"/>
       <dynamics damping="0.2"/>
@@ -87,5 +87,5 @@
       <parent link="base_link"/>
       <child link="right_wheel"/>
-      <origin xyz=".22 -.29 ${z_offset}" rpy="0 0 0"/>
+      <origin xyz="0 -.29 ${z_offset}" rpy="0 0 0"/>
       <axis xyz="0 1 0"/>
       <dynamics damping="0.2"/>

Commit message: update URDF
now robot wheel base is properly aligned with 0

File: src/IIR_base/urdf/iir_description.urdf.xacro (robot description, xacro)
@@ -17,7 +17,7 @@
   <!-- Base Link -->
   <link name="base_link">
-  <origin xyz="-0.1 0 0"/>
+  <origin xyz="-0.13 0 0"/>
     <collision>
-      <origin xyz="0 0 ${base_height/2}" rpy="0 0 0"/>
+      <origin xyz="-.13 0 ${base_height/2}" rpy="0 0 0"/>
       <geometry>
         <box size="${base_width} ${base_length} ${base_height}"/>

Commit message: change urdf for proper wheel seps and radius

File: src/IIR_base/urdf/iir_description.urdf.xacro (robot description, xacro)
@@ -11,5 +11,5 @@
   <xacro:property name="wheel_len" value="0.040" />
   <!-- wheels are .5m apart -->
-  <xacro:property name="wheel_radius" value="0.05" />
+  <xacro:property name="wheel_radius" value="0.0635" />
   <xacro:property name="caster_wheel_mass" value="0.1" /> <!-- arbitrary value for caster wheel mass -->
   <xacro:property name="caster_wheel_radius" value="0.042" />

File: src/IIR_base/urdf/iirbot.ros2_control.xacro (robot description, xacro)
@@ -43,6 +43,6 @@
   <right_joint>right_wheel_joint</right_joint>
   <!-- kinematics -->
-  <wheel_separation>0.48</wheel_separation>
-  <wheel_radius>0.05</wheel_radius> <!-- computed from <wheel_diameter> in the original plugin-->
+  <wheel_separation>.508</wheel_separation>
+  <wheel_radius>0.0635</wheel_radius> <!-- computed from <wheel_diameter> in the original plugin-->
   <!-- limits -->
   <max_linear_acceleration>100</max_linear_acceleration> <!-- computed from <max_linear_acceleration> in the original plugin-->

Commit message: add base_footprint for nav2

File: src/IIR_base/urdf/iir_description.urdf.xacro (robot description, xacro)
@@ -174,4 +174,9 @@
       </link>
       -->
+    <joint name="base_link_joint" type="fixed">
+  <parent link="base_footprint"/>
+  <child link="base_link"/>
+  <origin xyz="0 0 0.05" rpy="0 0 0"/>
+</joint>
     <joint name="caster_rear_wheel_joint" type="fixed">
       <parent link="base_link"/>

Commit message: try removing the params asking for base_footprint

File: src/IIR_base/urdf/iir_description.urdf.xacro (robot description, xacro)
@@ -174,10 +174,4 @@
       </link>
       -->
-      <link name="base_footprint" />
-    <joint name="base_link_joint" type="fixed">
-  <parent link="base_footprint"/>
-  <child link="base_link"/>
-  <origin xyz="0 0 0.05" rpy="0 0 0"/>
-</joint>
     <joint name="caster_rear_wheel_joint" type="fixed">
       <parent link="base_link"/>

Commit message: Update iir_description.urdf.xacro
rotate imus

File: src/IIR_base/urdf/iir_description.urdf.xacro (robot description, xacro)
@@ -78,9 +78,9 @@
       <parent link="base_link"/>
       <child link="imu_link_1"/>
-      <origin xyz="-0.35 -.20 ${base_height}" rpy="0 0 0"/>
+      <origin xyz="-0.35 -.20 ${base_height}" rpy="0 0 -${PI/2}"/>
     </joint>
     <link name="imu_link_1">
       <inertial>
-        <origin xyz="0 0 0" rpy="0 0 0"/>
+        <origin xyz="0 0 0" rpy="0 0 -${PI/2}"/>
         <mass value="0.01"/>
         <inertia
@@ -91,12 +91,12 @@
     </link>
  <!-- IMU Link -->
-    <joint name="imu_joint_2" type="fixed">
-      <parent link="base_link"/>
-      <child link="imu_link_2"/>
-      <origin xyz="-0.35 .20 ${base_height}" rpy="0 0 0"/>
-    </joint>
+  <joint name="imu_joint_2" type="fixed">
+    <parent link="base_link"/>
+    <child link="imu_link_2"/>
+    <origin xyz="-0.35 .20 ${base_height}" rpy="0 0 -${PI/2}"/>
+  </joint>
     <link name="imu_link_2">
       <inertial>
-        <origin xyz="0 0 0" rpy="0 0 0"/>
+        <origin xyz="0 0 0" rpy="0 0 -${PI/2}"/>
         <mass value="0.01"/>
         <inertia

Commit message: Update iir_description.urdf.xacro
rotate imus properly, i mounted differently than planned.

File: src/IIR_base/urdf/iir_description.urdf.xacro (robot description, xacro)
@@ -78,9 +78,9 @@
       <parent link="base_link"/>
       <child link="imu_link_1"/>
-      <origin xyz="-0.35 -.20 ${base_height}" rpy="0 0 -${PI/2}"/>
+      <origin xyz="-0.35 -.20 ${base_height}" rpy="0 0 ${PI/2}"/>
     </joint>
     <link name="imu_link_1">
       <inertial>
-        <origin xyz="0 0 0" rpy="0 0 -${PI/2}"/>
+        <origin xyz="0 0 0" rpy="0 0 ${PI/2}"/>
         <mass value="0.01"/>
         <inertia
@@ -94,9 +94,9 @@
     <parent link="base_link"/>
     <child link="imu_link_2"/>
-    <origin xyz="-0.35 .20 ${base_height}" rpy="0 0 -${PI/2}"/>
+    <origin xyz="-0.35 .20 ${base_height}" rpy="0 0 ${PI/2}"/>
   </joint>
     <link name="imu_link_2">
       <inertial>
-        <origin xyz="0 0 0" rpy="0 0 -${PI/2}"/>
+        <origin xyz="0 0 0" rpy="0 0 ${PI/2}"/>
         <mass value="0.01"/>
         <inertia

Commit message: update imu topic numbers
for clarity, rename 2 to 1, and 1 to 0. this lines up with how they must be declared in ekf.yaml.

File: src/IIR_base/urdf/iir_description.urdf.xacro (robot description, xacro)
@@ -75,10 +75,10 @@
       </link>
  <!-- IMU Link -->
-    <joint name="imu_joint_1" type="fixed">
-      <parent link="base_link"/>
-      <child link="imu_link_1"/>
+    <joint name="imu_joint_0" type="fixed">
+      <parent link="base_link"/>
+      <child link="imu_link_0"/>
       <origin xyz="-0.35 -.20 ${base_height}" rpy="0 0 ${PI/2}"/>
     </joint>
-    <link name="imu_link_1">
+    <link name="imu_link_0">
       <inertial>
         <origin xyz="0 0 0" rpy="0 0 ${PI/2}"/>
@@ -91,10 +91,10 @@
     </link>
  <!-- IMU Link -->
-  <joint name="imu_joint_2" type="fixed">
+  <joint name="imu_joint_1" type="fixed">
     <parent link="base_link"/>
-    <child link="imu_link_2"/>
+    <child link="imu_link_1"/>
     <origin xyz="-0.35 .20 ${base_height}" rpy="0 0 ${PI/2}"/>
   </joint>
-    <link name="imu_link_2">
+    <link name="imu_link_1">
       <inertial>
         <origin xyz="0 0 0" rpy="0 0 ${PI/2}"/>

Commit message: add pointcloud->scan package, add depth camera link

File: src/IIR_base/urdf/iir_description.urdf.xacro (robot description, xacro)
@@ -226,4 +226,40 @@
         </inertial>
       </link>
+    <!-- Depth Camera Link -->
+    <joint name="depth_camera_joint" type="fixed">
+      <parent link="base_link"/>
+      <child link="depth_camera_link"/>
+      <origin xyz="0.14 0 ${base_height}" rpy="0 0 0"/>
+    </joint>
+    <link name="depth_camera_link">
+      <visual>
+        <origin xyz="0 0 0" rpy="0 0 0"/>
+        <geometry>
+          <box size="0.025 0.09 0.025"/>
+        </geometry>
+        <material name="black"/>
+      </visual>
+      <collision>
+        <origin xyz="0 0 0" rpy="0 0 0"/>
+        <geometry>
+          <box size="0.025 0.09 0.025"/>
+        </geometry>
+      </collision>
+      <inertial>
+        <origin xyz="0 0 0" rpy="0 0 0"/>
+        <mass value="0.05"/>
+        <inertia
+          ixx="0.0001" ixy="0.0" ixz="0.0"
+          iyy="0.0001" iyz="0.0"
+          izz="0.0001"/>
+      </inertial>
+    </link>
+    <!-- Depth Camera Optical Frame (ROS convention: z forward, x right, y down) -->
+    <joint name="depth_camera_optical_joint" type="fixed">
+      <parent link="depth_camera_link"/>
+      <child link="depth_camera_optical_frame"/>
+      <origin xyz="0 0 0" rpy="${-PI/2} 0 ${-PI/2}"/>
+    </joint>
+    <link name="depth_camera_optical_frame"/>
   </xacro:macro>
 </robot>

Commit message: add is_on_wall launch arg
rotates the IMU urdf if we are on the wall

File: src/IIR_base/urdf/iir_description.urdf.xacro (robot description, xacro)
@@ -1,5 +1,5 @@
 <?xml version="1.0"?>
 <robot xmlns:xacro="http://www.ros.org/wiki/xacro">
-  <xacro:macro name="iirbot_desc" params="prefix">
+  <xacro:macro name="iirbot_desc" params="prefix is_on_wall">
   <!-- Constants for robot dimensions -->
   <xacro:property name="PI" value="3.1415926535897931"/>
@@ -75,12 +75,24 @@
       </link>
  <!-- IMU Link -->
+<!-- in the future, we could look into changing these joint types to resolute or floating, and update the imu's rotation based off of its quaternion output -->
+<!-- This may allow for better modeling of the robots behaviour in 3D space. -->
     <joint name="imu_joint_0" type="fixed">
       <parent link="base_link"/>
       <child link="imu_link_0"/>
-      <origin xyz="-0.35 -.20 ${base_height}" rpy="0 0 ${PI/2}"/>
+        <xacro:if value="${is_on_wall}">
+          <origin xyz="-0.35 .20 ${base_height}" rpy="${PI/2} 0 ${PI/2}"/>
+        </xacro:if>
+        <xacro:unless value="${is_on_wall}">
+        <origin xyz="-0.35 -.20 ${base_height}" rpy="0 0 ${PI/2}"/>
+        </xacro:unless>
     </joint>
     <link name="imu_link_0">
       <inertial>
-        <origin xyz="0 0 0" rpy="0 0 ${PI/2}"/>
+        <xacro:if value="${is_on_wall}">
+          <origin xyz="0 0 0" rpy="${PI/2} 0 ${PI/2}"/>
+        </xacro:if>
+        <xacro:unless value="${is_on_wall}">
+          <origin xyz="0 0 0" rpy="0 0 ${PI/2}"/>
+        </xacro:unless>
         <mass value="0.01"/>
         <inertia
@@ -94,9 +106,19 @@
     <parent link="base_link"/>
     <child link="imu_link_1"/>
+    <xacro:if value="${is_on_wall}">
+      <origin xyz="-0.35 -.20 ${base_height}" rpy="${PI/2} 0 ${PI/2}"/>
+    </xacro:if>
+    <xacro:unless value="${is_on_wall}">
     <origin xyz="-0.35 .20 ${base_height}" rpy="0 0 ${PI/2}"/>
+    </xacro:unless>
   </joint>
     <link name="imu_link_1">
       <inertial>
-        <origin xyz="0 0 0" rpy="0 0 ${PI/2}"/>
+        <xacro:if value="${is_on_wall}">
+          <origin xyz="0 0 0" rpy="${PI/2} 0 ${PI/2}"/>
+        </xacro:if>
+        <xacro:unless value="${is_on_wall}">
+          <origin xyz="0 0 0" rpy="0 0 ${PI/2}"/>
+        </xacro:unless>
         <mass value="0.01"/>
         <inertia

File: src/IIR_base/urdf/iirbot.urdf.xacro (robot description, xacro)
@@ -4,4 +4,5 @@
   <xacro:arg name="prefix" default="" />
   <xacro:arg name="use_mock_hardware" default="false" />
+  <xacro:arg name="is_on_wall" default="false" />
   <xacro:include filename="$(find iir_base)/urdf/iir_description.urdf.xacro" />
   <!-- Import Rviz colors -->
@@ -10,5 +11,5 @@
   <!-- Import diffbot ros2_control description -->
   <xacro:include filename="$(find iir_base)/urdf/iirbot.ros2_control.xacro" />
-  <xacro:iirbot_desc prefix="$(arg prefix)" />
+  <xacro:iirbot_desc prefix="$(arg prefix)" is_on_wall="$(arg is_on_wall)" />
   <xacro:hokuyo_ust10_mount prefix="" topic="scan" parent_link="base_link" min_angle="-2.35619" max_angle="2.35619">
   <origin xyz="0 0 0.1" rpy="0 0 0" />
